File: light/light.sch (KiCad schematic (older format))
At the start: 8 parts

Commit message: Second commit
Parts:
- removed R?: R, symbol device:R
- added D1: 1N4148, Diodes_THT:D_DO-35_SOD27_P7.62mm_Horizontal, symbol Diode:1N4148
- added R2: 1k, symbol device:R
- J1: renamed from J?; footprint (none) -> Pin_Headers:Pin_Header_Straight_2x03_Pitch2.54mm
- gave numbers to parts that had none: 6
Connections:
- wire segments 40 -> 45
Changed lines of the file:
@@
 $EndDescr
 $Comp
-L atmel:ATMEGA8-16AU U?
+L atmel:ATMEGA8-16AU U1
 U 1 1 5A32B259
 P 6000 3550
-F 0 "U?" H 5300 4750 50  0000 C CNN
+F 0 "U1" H 5300 4750 50  0000 C CNN
 F 1 "ATMEGA8-16AU" H 6550 4750 50  0000 C CNN
 F 2 "Housings_QFP:LQFP-32_7x7mm_Pitch0.8mm" H 6000 3550 50  0001 C CIN
@@
 $EndComp
 $Comp
-L device:R R?
-U 1 1 5A32B317
-P 3900 1500
-F 0 "R?" H 3970 1546 50  0000 L CNN
-F 1 "R" H 3970 1455 50  0000 L CNN
-F 2 "" V 3830 1500 50  0001 C CNN
-F 3 "" H 3900 1500 50  0001 C CNN
-	1    3900 1500
-	1    0    0    -1
-$EndComp
-$Comp
-L device:R R?
+L device:R R1
 U 1 1 5A32B3B5
 P 5550 2200
-F 0 "R?" V 5650 2150 50  0000 L CNN
+F 0 "R1" V 5650 2150 50  0000 L CNN
 F 1 "10k" V 5450 2100 50  0000 L CNN
 F 2 "" V 5480 2200 50  0001 C CNN
@@
 $EndComp
 $Comp
-L power:GND #PWR?
+L power:GND #PWR07
 U 1 1 5A32B471
 P 5950 5250
-F 0 "#PWR?" H 5950 5000 50  0001 C CNN
+F 0 "#PWR07" H 5950 5000 50  0001 C CNN
 F 1 "GND" H 5955 5077 50  0000 C CNN
 F 2 "" H 5950 5250 50  0001 C CNN
@@
 $EndComp
 $Comp
-L power:GND #PWR?
+L power:GND #PWR09
 U 1 1 5A32B4B1
 P 6050 5250
-F 0 "#PWR?" H 6050 5000 50  0001 C CNN
+F 0 "#PWR09" H 6050 5000 50  0001 C CNN
 F 1 "GND" H 6055 5077 50  0000 C CNN
 F 2 "" H 6050 5250 50  0001 C CNN
@@
 	5950 5250 5950 5150
 $Comp
-L power:PWR_FLAG #FLG?
+L power:PWR_FLAG #FLG01
 U 1 1 5A32B54C
 P 8450 1250
-F 0 "#FLG?" H 8450 1325 50  0001 C CNN
+F 0 "#FLG01" H 8450 1325 50  0001 C CNN
 F 1 "PWR_FLAG" H 8450 1424 50  0000 C CNN
 F 2 "" H 8450 1250 50  0001 C CNN
@@
 $EndComp
 $Comp
-L power:PWR_FLAG #FLG?
+L power:PWR_FLAG #FLG02
 U 1 1 5A32B56D
 P 8900 1250
-F 0 "#FLG?" H 8900 1325 50  0001 C CNN
+F 0 "#FLG02" H 8900 1325 50  0001 C CNN
 F 1 "PWR_FLAG" H 8900 1424 50  0000 C CNN
 F 2 "" H 8900 1250 50  0001 C CNN
@@
 $EndComp
 $Comp
-L power:GND #PWR?
+L power:GND #PWR012
 U 1 1 5A32B58D
 P 8450 1450
-F 0 "#PWR?" H 8450 1200 50  0001 C CNN
+F 0 "#PWR012" H 8450 1200 50  0001 C CNN
 F 1 "GND" H 8455 1277 50  0000 C CNN
 F 2 "" H 8450 1450 50  0001 C CNN
@@
 	8450 1450 8450 1250
 $Comp
-L Connector:Conn_01x06 J?
+L Connector:Conn_01x06 J1
 U 1 1 5A347467
 P 9600 3250
-F 0 "J?" H 9680 3242 50  0000 L CNN
+F 0 "J1" H 9680 3242 50  0000 L CNN
 F 1 "AVR_SPI" H 9680 3151 50  0000 L CNN
-F 2 "" H 9600 3250 50  0001 C CNN
+F 2 "Pin_Headers:Pin_Header_Straight_2x03_Pitch2.54mm" H 9600 3250 50  0001 C CNN
 F 3 "~" H 9600 3250 50  0001 C CNN
 	1    9600 3250
@@
 RES
 $Comp
-L power:GND #PWR?
+L power:GND #PWR015
 U 1 1 5A347606
 P 9300 3650
-F 0 "#PWR?" H 9300 3400 50  0001 C CNN
+F 0 "#PWR015" H 9300 3400 50  0001 C CNN
 F 1 "GND" H 9305 3477 50  0000 C CNN
 F 2 "" H 9300 3650 50  0001 C CNN
@@
 	9300 3550 9400 3550
 $Comp
-L power:VCC #PWR?
+L power:VCC #PWR06
 U 1 1 5A3476ED
 P 5950 2150
-F 0 "#PWR?" H 5950 2000 50  0001 C CNN
+F 0 "#PWR06" H 5950 2000 50  0001 C CNN
 F 1 "VCC" H 5900 2300 50  0000 C CNN
 F 2 "" H 5950 2150 50  0001 C CNN
@@
 $EndComp
 $Comp
-L power:VCC #PWR?
+L power:VCC #PWR08
 U 1 1 5A347717
 P 6050 2150
-F 0 "#PWR?" H 6050 2000 50  0001 C CNN
+F 0 "#PWR08" H 6050 2000 50  0001 C CNN
 F 1 "VCC" H 6100 2300 50  0000 C CNN
 F 2 "" H 6050 2150 50  0001 C CNN
@@
 	5950 2150 5950 2200
 $Comp
-L power:VCC #PWR?
+L power:VCC #PWR013
 U 1 1 5A3479D0
 P 9050 3050
-F 0 "#PWR?" H 9050 2900 50  0001 C CNN
+F 0 "#PWR013" H 9050 2900 50  0001 C CNN
 F 1 "VCC" H 9100 3200 50  0000 C CNN
 F 2 "" H 9050 3050 50  0001 C CNN
@@
 	5950 2200 5950 2250
 $Comp
-L device:C C?
+L device:C C1
 U 1 1 5A348923
 P 4450 2200
-F 0 "C?" V 4198 2200 50  0000 C CNN
+F 0 "C1" V 4198 2200 50  0000 C CNN
 F 1 "100n" V 4289 2200 50  0000 C CNN
 F 2 "" H 4488 2050 50  0001 C CNN
@@
 $EndComp
 $Comp
-L power:GND #PWR?
+L power:GND #PWR01
 U 1 1 5A348C8E
 P 4150 2200
-F 0 "#PWR?" H 4150 1950 50  0001 C CNN
+F 0 "#PWR01" H 4150 1950 50  0001 C CNN
 F 1 "GND" H 4155 2027 50  0000 C CNN
 F 2 "" H 4150 2200 50  0001 C CNN
@@
 	4950 2200 5400 2200
 $Comp
-L power:VCC #PWR?
+L power:VCC #PWR03
 U 1 1 5A365230
 P 4750 2600
-F 0 "#PWR?" H 4750 2450 50  0001 C CNN
+F 0 "#PWR03" H 4750 2450 50  0001 C CNN
 F 1 "VCC" H 4800 2750 50  0000 C CNN
 F 2 "" H 4750 2600 50  0001 C CNN
@@
 	4750 2750 5100 2750
 $Comp
-L power:GND #PWR?
+L power:GND #PWR04
 U 1 1 5A365567
 P 4850 2950
-F 0 "#PWR?" H 4850 2700 50  0001 C CNN
+F 0 "#PWR04" H 4850 2700 50  0001 C CNN
 F 1 "GND" H 4855 2777 50  0000 C CNN
 F 2 "" H 4850 2950 50  0001 C CNN
@@
 	4850 2950 5100 2950
 $Comp
-L device:Crystal Y?
+L device:Crystal Y1
 U 1 1 5A3659C3
 P 4800 3450
-F 0 "Y?" H 4650 3500 50  0000 C CNN
+F 0 "Y1" H 4650 3500 50  0000 C CNN
 F 1 "9.261Mhz" H 4800 3300 50  0000 C CNN
 F 2 "" H 4800 3450 50  0001 C CNN
@@
 	5100 3450 5050 3450
 $Comp
-L device:C C?
+L device:C C2
 U 1 1 5A36641A
 P 4500 3800
-F 0 "C?" H 4615 3846 50  0000 L CNN
+F 0 "C2" H 4615 3846 50  0000 L CNN
 F 1 "22p" H 4615 3755 50  0000 L CNN
 F 2 "" H 4538 3650 50  0001 C CNN
@@
 $EndComp
 $Comp
-L device:C C?
+L device:C C3
 U 1 1 5A36649F
 P 5050 3800
-F 0 "C?" H 5165 3846 50  0000 L CNN
+F 0 "C3" H 5165 3846 50  0000 L CNN
 F 1 "22p" H 5165 3755 50  0000 L CNN
 F 2 "" H 5088 3650 50  0001 C CNN
@@
 $EndComp
 $Comp
-L power:GND #PWR?
+L power:GND #PWR02
 U 1 1 5A3664E2
 P 4500 4050
-F 0 "#PWR?" H 4500 3800 50  0001 C CNN
+F 0 "#PWR02" H 4500 3800 50  0001 C CNN
 F 1 "GND" H 4505 3877 50  0000 C CNN
 F 2 "" H 4500 4050 50  0001 C CNN
@@
 $EndComp
 $Comp
-L power:GND #PWR?
+L power:GND #PWR05
 U 1 1 5A366515
 P 5050 4050
-F 0 "#PWR?" H 5050 3800 50  0001 C CNN
+F 0 "#PWR05" H 5050 3800 50  0001 C CNN
 F 1 "GND" H 5055 3877 50  0000 C CNN
 F 2 "" H 5050 4050 50  0001 C CNN
@@
 	5050 3450 4950 3450
 $Comp
-L power:VCC #PWR?
+L power:VCC #PWR014
 U 1 1 5A367BBB
 P 9300 1250
-F 0 "#PWR?" H 9300 1100 50  0001 C CNN
+F 0 "#PWR014" H 9300 1100 50  0001 C CNN
 F 1 "VCC" H 9350 1400 50  0000 C CNN
 F 2 "" H 9300 1250 50  0001 C CNN
@@
 Text Label 7200 4250 0    60   ~ 0
 RX
+$Comp
+L Diode:1N4148 D1
+U 1 1 5A369509
+P 8000 3450
+F 0 "D1" V 7954 3529 50  0000 L CNN
+F 1 "1N4148" V 8045 3529 50  0000 L CNN
+F 2 "Diodes_THT:D_DO-35_SOD27_P7.62mm_Horizontal" H 8000 3275 50  0001 C CNN
+F 3 "http://www.nxp.com/documents/data_sheet/1N4148_1N4448.pdf" H 8000 3450 50  0001 C CNN
+	1    8000 3450
+	0    1    1    0
+$EndComp
+$Comp
+L power:GND #PWR011
+U 1 1 5A36958B
+P 8000 3700
+F 0 "#PWR011" H 8000 3450 50  0001 C CNN
+F 1 "GND" H 8005 3527 50  0000 C CNN
+F 2 "" H 8000 3700 50  0001 C CNN
+F 3 "" H 8000 3700 50  0001 C CNN
+	1    8000 3700
+	1    0    0    -1
+$EndComp
+Wire Wire Line
+	8000 3700 8000 3600
+$Comp
+L device:R R2
+U 1 1 5A369DDB
+P 8000 3000
+F 0 "R2" H 8070 3046 50  0000 L CNN
+F 1 "1k" H 8070 2955 50  0000 L CNN
+F 2 "" V 7930 3000 50  0001 C CNN
+F 3 "" H 8000 3000 50  0001 C CNN
+	1    8000 3000
+	1    0    0    -1
+$EndComp
+Wire Wire Line
+	8000 3300 8000 3250
+Wire Wire Line
+	7000 3250 8000 3250
+Connection ~ 8000 3250
+Wire Wire Line
+	8000 3250 8000 3150
+$Comp
+L power:VCC #PWR010
+U 1 1 5A36AF04
+P 8000 2750
+F 0 "#PWR010" H 8000 2600 50  0001 C CNN
+F 1 "VCC" H 8050 2900 50  0000 C CNN
+F 2 "" H 8000 2750 50  0001 C CNN
+F 3 "" H 8000 2750 50  0001 C CNN
+	1    8000 2750
+	1    0    0    -1
+$EndComp
+Wire Wire Line
+	8000 2750 8000 2850
 $EndSCHEMATC

Commit message: Test uart tx
Parts:
- removed U1: ATMEGA8-16AU, Housings_QFP:LQFP-32_7x7mm_Pitch0.8mm, symbol atmel:ATMEGA8-16AU
- added U1: ATMEGA8-16PU, Housings_DIP:DIP-28_W7.62mm, symbol atmel:ATMEGA8-16PU
Connections:
- wire segments 45 -> 43

Commit message: Add temperature measure
Parts:
- added C?: 100n, symbol light-rescue:C-device
- added U?: ATMEGA16-16AU, TQFP44, symbol MCU_Atmel_ATMEGA:ATMEGA16-16AU
- C1, C2, C3: symbol device:C -> light-rescue:C-device
- J1: symbol Connector:Conn_01x06 -> light-rescue:Conn_01x06-Connector
- R1, R2: symbol device:R -> light-rescue:R-device
- U1: symbol atmel:ATMEGA8-16PU -> light-rescue:ATMEGA8-16PU-atmel
- Y1: symbol device:Crystal -> light-rescue:Crystal-device
Connections:
- wire segments 43 -> 46
Changed lines of the file:
@@
 $EndDescr
 $Comp
-L device:R R1
+L light-rescue:R-device R1
 U 1 1 5A32B3B5
 P 2700 1100
@@
 	4350 1050 4350 850
 $Comp
-L Connector:Conn_01x06 J1
+L light-rescue:Conn_01x06-Connector J1
 U 1 1 5A347467
 P 5700 2200
@@
 	3150 1100 3150 1150
 $Comp
-L device:C C1
+L light-rescue:C-device C1
 U 1 1 5A348923
 P 1600 1100
@@
 	2000 1850 2250 1850
 $Comp
-L device:Crystal Y1
+L light-rescue:Crystal-device Y1
 U 1 1 5A3659C3
 P 1950 2350
@@
 	2250 2350 2200 2350
 $Comp
-L device:C C2
+L light-rescue:C-device C2
 U 1 1 5A36641A
 P 1650 2700
@@
 $EndComp
 $Comp
-L device:C C3
+L light-rescue:C-device C3
 U 1 1 5A36649F
 P 2200 2700
@@
 $EndComp
 $Comp
-L device:R R2
+L light-rescue:R-device R2
 U 1 1 5A369DDB
 P 4750 1900
@@
 	4750 1650 4750 1750
 $Comp
-L atmel:ATMEGA8-16PU U1
+L light-rescue:ATMEGA8-16PU-atmel U1
 U 1 1 5A343891
 P 3150 2550
@@
 	4750 2250 4750 2150
 Connection ~ 4750 2150
+$Comp
+L MCU_Atmel_ATMEGA:ATMEGA16-16AU U?
+U 1 1 5A6664FD
+P 8000 3050
+F 0 "U?" H 8000 5228 50  0000 C CNN
+F 1 "ATMEGA16-16AU" H 8000 5137 50  0000 C CNN
+F 2 "TQFP44" H 8000 3050 50  0001 C CIN
+F 3 "http://ww1.microchip.com/downloads/en/DeviceDoc/doc2466.pdf" H 8000 3050 50  0001 C CNN
+	1    8000 3050
+	1    0    0    -1
+$EndComp
+$Comp
+L light-rescue:C-device C?
+U 1 1 5A666732
+P 1350 2050
+F 0 "C?" H 1465 2096 50  0000 L CNN
+F 1 "100n" H 1465 2005 50  0000 L CNN
+F 2 "" H 1388 1900 50  0001 C CNN
+F 3 "" H 1350 2050 50  0001 C CNN
+	1    1350 2050
+	1    0    0    -1
+$EndComp
+Wire Wire Line
+	1350 1750 2250 1750
+Wire Wire Line
+	1350 1750 1350 1900
+$Comp
+L power:GND #PWR?
+U 1 1 5A667154
+P 1350 2350
+F 0 "#PWR?" H 1350 2100 50  0001 C CNN
+F 1 "GND" H 1355 2177 50  0000 C CNN
+F 2 "" H 1350 2350 50  0001 C CNN
+F 3 "" H 1350 2350 50  0001 C CNN
+	1    1350 2350
+	1    0    0    -1
+$EndComp
+Wire Wire Line
+	1350 2350 1350 2200
 $EndSCHEMATC
